Commit message: Update camera to the bot and read camera data

File: urdf/ackermann_bot.urdf.xacro (robot description, xacro)
@@ -105,4 +105,31 @@
   <xacro:rear_wheel wheel_name="rear_left_wheel" y_offset="${wheel_offset_y}"/>
   <xacro:rear_wheel wheel_name="rear_right_wheel" y_offset="-${wheel_offset_y}"/>
+  <!-- Camera Link -->
+  <link name="camera_link">
+    <visual>
+      <origin xyz="0 0 0" rpy="0 0 0"/>
+      <geometry>
+        <box size="0.03 0.03 0.02"/>
+      </geometry>
+      <material name="blue"/>
+    </visual>
+    <collision>
+      <origin xyz="0 0 0" rpy="0 0 0"/>
+      <geometry>
+        <box size="0.03 0.03 0.02"/>
+      </geometry>
+    </collision>
+    <inertial>
+      <origin xyz="0 0 0" rpy="0 0 0"/>
+      <mass value="0.05"/>
+      <xacro:box_inertia m="0.05" l="0.03" w="0.03" h="0.02"/>
+    </inertial>
+  </link>
+  <!-- Camera Joint -->
+  <joint name="camera_joint" type="fixed">
+    <parent link="base_link"/>
+    <child link="camera_link"/>
+    <origin xyz="${chassis_length/2} 0 ${chassis_height + 0.05}" rpy="0 0 0"/>
+  </joint>
   <!-- Gazebo Ackermann steering plugin -->
   <gazebo>
@@ -137,4 +164,7 @@
     <material>Gazebo/Red</material>
   </gazebo>
+  <gazebo reference="camera_link">
+    <material>Gazebo/Blue</material>
+  </gazebo>
   <gazebo reference="front_left_wheel">
     <material>Gazebo/DarkGrey</material>
@@ -149,3 +179,25 @@
     <material>Gazebo/DarkGrey</material>
   </gazebo>
+  <!-- Camera sensor -->
+  <gazebo reference="camera_link">
+    <sensor name="camera_sensor" type="camera">
+      <update_rate>10</update_rate>
+      <visualize>true</visualize>
+      <camera name="camera">
+        <horizontal_fov>1.0472</horizontal_fov>
+        <image>
+          <width>640</width>
+          <height>480</height>
+          <format>R8G8B8</format>
+        </image>
+        <clip>
+          <near>0.1</near>
+          <far>100</far>
+        </clip>
+      </camera>
+      <plugin filename="gz-sim-sensors-system" name="gz::sim::systems::Sensors">
+        <render_engine>ogre2</render_engine>
+      </plugin>
+    </sensor>
+  </gazebo>
 </robot>

Commit message: dev-lidar add lidar sensor to out bot, add check lidar topics and lidar test for reading lidar data

File: urdf/ackermann_bot.urdf.xacro (robot description, xacro)
@@ -132,4 +132,31 @@
     <origin xyz="${chassis_length/2} 0 ${chassis_height + 0.05}" rpy="0 0 0"/>
   </joint>
+  <!-- Lidar Link -->
+  <link name="lidar_link">
+    <visual>
+      <origin xyz="0 0 0" rpy="0 0 0"/>
+      <geometry>
+        <cylinder radius="0.05" length="0.04"/>
+      </geometry>
+      <material name="black"/>
+    </visual>
+    <collision>
+      <origin xyz="0 0 0" rpy="0 0 0"/>
+      <geometry>
+        <cylinder radius="0.05" length="0.04"/>
+      </geometry>
+    </collision>
+    <inertial>
+      <origin xyz="0 0 0" rpy="0 0 0"/>
+      <mass value="0.1"/>
+      <xacro:cylinder_inertia m="0.1" r="0.05" h="0.04"/>
+    </inertial>
+  </link>
+  <!-- Lidar Joint -->
+  <joint name="lidar_joint" type="fixed">
+    <parent link="base_link"/>
+    <child link="lidar_link"/>
+    <origin xyz="0 0 ${chassis_height + 0.08}" rpy="0 0 0"/>
+  </joint>
   <!-- Gazebo Ackermann steering plugin -->
   <gazebo>
@@ -155,4 +182,10 @@
     </plugin>
   </gazebo>
+  <!-- Global Sensors System Plugin (must be defined once globally) -->
+  <gazebo>
+    <plugin filename="gz-sim-sensors-system" name="gz::sim::systems::Sensors">
+      <render_engine>ogre2</render_engine>
+    </plugin>
+  </gazebo>
   <!-- Joint state publisher plugin -->
   <gazebo>
@@ -166,4 +199,7 @@
   <gazebo reference="camera_link">
     <material>Gazebo/Blue</material>
+  </gazebo>
+  <gazebo reference="lidar_link">
+    <material>Gazebo/Black</material>
   </gazebo>
   <gazebo reference="front_left_wheel">
@@ -196,8 +232,39 @@
         </clip>
       </camera>
-      <plugin filename="gz-sim-sensors-system" name="gz::sim::systems::Sensors">
-        <render_engine>ogre2</render_engine>
-      </plugin>
     </sensor>
   </gazebo>
+  <!-- Lidar sensor -->
+  <gazebo reference="lidar_link">
+    <sensor name="lidar_sensor" type="gpu_lidar">
+      <update_rate>10</update_rate>
+      <visualize>true</visualize>
+      <always_on>true</always_on>
+      <lidar>
+        <scan>
+          <horizontal>
+            <samples>360</samples>
+            <resolution>1</resolution>
+            <min_angle>-3.141592</min_angle>
+            <max_angle>3.141592</max_angle>
+          </horizontal>
+          <vertical>
+            <samples>1</samples>
+            <resolution>1</resolution>
+            <min_angle>0</min_angle>
+            <max_angle>0</max_angle>
+          </vertical>
+        </scan>
+        <range>
+          <min>0.1</min>
+          <max>10.0</max>
+          <resolution>0.01</resolution>
+        </range>
+        <noise>
+          <type>gaussian</type>
+          <mean>0.0</mean>
+          <stddev>0.01</stddev>
+        </noise>
+      </lidar>
+    </sensor>
+  </gazebo>
 </robot>

Commit message: change to 2d lidar

File: urdf/ackermann_bot.urdf.xacro (robot description, xacro)
@@ -185,5 +185,5 @@
   <gazebo>
     <plugin filename="gz-sim-sensors-system" name="gz::sim::systems::Sensors">
-      <render_engine>ogre2</render_engine>
+      <render_engine>${render_engine}</render_engine>
     </plugin>
   </gazebo>
@@ -234,7 +234,7 @@
     </sensor>
   </gazebo>
-  <!-- 3D Lidar sensor -->
+  <!-- Lidar sensor -->
   <gazebo reference="lidar_link">
-    <sensor name="lidar_sensor" type="gpu_lidar">
+    <sensor name="lidar_sensor" type="${lidar_type}">
       <update_rate>10</update_rate>
       <visualize>true</visualize>
@@ -244,13 +244,13 @@
           <horizontal>
             <samples>360</samples>
-            <resolution>0.5</resolution>
+            <resolution>1</resolution>
             <min_angle>-3.141592</min_angle>
             <max_angle>3.141592</max_angle>
           </horizontal>
           <vertical>
-            <samples>64</samples>
-            <resolution>0.5</resolution>
-            <min_angle>-0.419</min_angle>
-            <max_angle>0.419</max_angle>
+            <samples>1</samples>
+            <resolution>1</resolution>
+            <min_angle>0</min_angle>
+            <max_angle>0</max_angle>
           </vertical>
         </scan>

File: urdf/properties.xacro (robot description, xacro)
@@ -25,3 +25,7 @@
              izz="${m*r*r/2}"/>
   </xacro:macro>
+  <!-- Lidar type - can be 'gpu_lidar' or 'lidar' -->
+  <xacro:property name="lidar_type" value="gpu_lidar"/>
+    <!-- Render Engine Type - can be 'ogre' or 'ogre2' -->
+  <xacro:property name="render_engine" value="ogre2"/>
 </robot>
